File: eagle/ll_both.brd (EAGLE design)
At the start: 100 x 75 mm, 11 parts, among them U1 ATTINY45-20P

Commit message: first eagle pcb layout
Parts:
- removed PHOTO_ADC1: (no value), jumper:JP1
- added C2: 100nF, rcl:C025-025X050
- added POWER1, POWER2: (no value), jumper:JP1
- moved BUTTON 39.7 mm to (7.62, 69.8)
- moved PHOTO_ADC 27.5 mm to (28.6, 67.3), turned to 0 degrees
- moved R_PHOTO 1.27 mm to (19.1, 51.4)
- moved RGB_LED 1.27 mm to (24.1, 42.5)
Connections:
- net GND: now also C2.2, POWER1.1, POWER2.1; no longer PHOTO_ADC1.1
- net VCC: now also C2.1, POWER1.2, POWER2.2; no longer PHOTO_ADC1.2
Routing:
- net N$8: track 90.8 -> 12.1 mm, vias 2 -> 0
- net GND: track 105.3 -> 155.3 mm, vias 2 -> 0
- net VCC: track 70.4 -> 89.5 mm, vias 0 -> 2
- net MOSI: track 35.7 -> 46.6 mm, vias 2 -> 0
- net SCK: track 47.0 -> 40.9 mm
- net N$5: track 0.00 -> 2.54 mm
- net RESET: track 25.5 -> 23.7 mm, vias 2 -> 0
- net N$6: track 35.9 -> 34.4 mm
- net N$4: track 4.97 -> 6.24 mm
- net N$2: track 3.81 -> 5.08 mm
- added copper zone on layer 16, net GND
Other:
- board text added: "LaserLabyrinth Test v0.1"
