File: eagle/ll_both.sch (EAGLE design)
At the start: 11 parts, among them U1 ATTINY45-20P

Commit message: first eagle pcb layout
Parts:
- added C2: 100nF, rcl:C-EU025-025X050
- added POWER1: (no value), jumper:JP1E
- renumbered PHOTO_ADC1 to POWER2
Connections:
- net GND: now also C2.2, POWER1.1
- net VCC: now also C2.1, POWER1.2
Changed lines of the file:
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@@
 <part name="P+3" library="supply1" deviceset="VCC" device=""/>
 <part name="GND6" library="supply1" deviceset="GND" device=""/>
-<part name="PHOTO_ADC1" library="jumper" deviceset="JP1E" device=""/>
+<part name="POWER2" library="jumper" deviceset="JP1E" device=""/>
 <part name="P+4" library="supply1" deviceset="VCC" device=""/>
 <part name="GND7" library="supply1" deviceset="GND" device=""/>
 <part name="U1" library="attiny25_45_85" deviceset="ATTINY45*" device="P" technology="-20"/>
+<part name="C2" library="rcl" deviceset="C-EU" device="025-025X050" value="100nF"/>
+<part name="POWER1" library="jumper" deviceset="JP1E" device=""/>
+<part name="GND8" library="supply1" deviceset="GND" device=""/>
+<part name="P+5" library="supply1" deviceset="VCC" device=""/>
 </parts>
 <sheets>
@@
 <instance part="P+3" gate="VCC" x="48.26" y="96.52" rot="R270"/>
 <instance part="GND6" gate="1" x="48.26" y="86.36" rot="R90"/>
-<instance part="PHOTO_ADC1" gate="A" x="99.06" y="27.94" rot="R270"/>
+<instance part="POWER2" gate="A" x="99.06" y="27.94" rot="R270"/>
 <instance part="P+4" gate="VCC" x="93.98" y="25.4" rot="R90"/>
 <instance part="GND7" gate="1" x="93.98" y="27.94" rot="R270"/>
 <instance part="U1" gate="G$1" x="25.4" y="58.42"/>
+<instance part="C2" gate="G$1" x="2.54" y="58.42"/>
+<instance part="POWER1" gate="A" x="111.76" y="27.94" rot="R270"/>
+<instance part="GND8" gate="1" x="104.14" y="27.94" rot="R270"/>
+<instance part="P+5" gate="VCC" x="104.14" y="25.4" rot="R90"/>
 </instances>
 <busses>
@@
 <segment>
 <pinref part="GND2" gate="1" pin="GND"/>
-<wire x1="0" y1="50.8" x2="10.16" y2="50.8" width="0.1524" layer="91"/>
+<wire x1="0" y1="50.8" x2="2.54" y2="50.8" width="0.1524" layer="91"/>
 <pinref part="U1" gate="G$1" pin="GND"/>
+<pinref part="C2" gate="G$1" pin="2"/>
+<wire x1="2.54" y1="50.8" x2="10.16" y2="50.8" width="0.1524" layer="91"/>
+<wire x1="2.54" y1="53.34" x2="2.54" y2="50.8" width="0.1524" layer="91"/>
 </segment>
 <segment>
@@
 </segment>
 <segment>
-<pinref part="PHOTO_ADC1" gate="A" pin="1"/>
+<pinref part="POWER2" gate="A" pin="1"/>
 <pinref part="GND7" gate="1" pin="GND"/>
+</segment>
+<segment>
+<pinref part="POWER1" gate="A" pin="1"/>
+<wire x1="109.22" y1="27.94" x2="106.68" y2="27.94" width="0.1524" layer="91"/>
+<pinref part="GND8" gate="1" pin="GND"/>
 </segment>
 </net>
@@
 <segment>
 <pinref part="P+1" gate="VCC" pin="VCC"/>
-<wire x1="-2.54" y1="63.5" x2="10.16" y2="63.5" width="0.1524" layer="91"/>
+<wire x1="-2.54" y1="63.5" x2="2.54" y2="63.5" width="0.1524" layer="91"/>
 <pinref part="U1" gate="G$1" pin="VCC"/>
+<pinref part="C2" gate="G$1" pin="1"/>
+<wire x1="2.54" y1="63.5" x2="10.16" y2="63.5" width="0.1524" layer="91"/>
+<wire x1="2.54" y1="60.96" x2="2.54" y2="63.5" width="0.1524" layer="91"/>
 </segment>
 <segment>
@@
 </segment>
 <segment>
-<pinref part="PHOTO_ADC1" gate="A" pin="2"/>
+<pinref part="POWER2" gate="A" pin="2"/>
 <pinref part="P+4" gate="VCC" pin="VCC"/>
 </segment>
+<segment>
+<pinref part="POWER1" gate="A" pin="2"/>
+<wire x1="109.22" y1="25.4" x2="106.68" y2="25.4" width="0.1524" layer="91"/>
+<pinref part="P+5" gate="VCC" pin="VCC"/>
+</segment>
 </net>
